File: IO.kicad_sch (KiCad schematic)
At the start: 22 parts

Commit message: Guardar cambios
Parts:
- removed 12VIN1: Conn_01x02, TerminalBlock_Phoenix:TerminalBlock_Phoenix_MKDS-1,5-2-5.08_1x02_P5.08mm_Horizontal, symbol Connector_Generic:Conn_01x02
- removed BUCK1: AP1509-50SG-13, Package_SO:SOP-8_3.76x4.96mm_P1.27mm, symbol AP1509:AP1509-50SG-13
- removed CIBUCK1, COBUCK1: C_Polarized, Capacitor_SMD:CP_Elec_8x6.2, symbol Device:C_Polarized
- removed CILDO1, COLDO1: C_Polarized, Capacitor_SMD:C_1206_3216Metric, symbol Device:C_Polarized
- removed CIN1: C, Capacitor_SMD:CP_Elec_8x6.2, symbol Device:C
- removed DBUCK1: B220, Diode_SMD:D_SMB, symbol Diode:B220
- removed FUENTE1, TIVA1: Conn_01x02, Connector_PinHeader_2.54mm:PinHeader_1x02_P2.54mm_Vertical, symbol Connector_Generic:Conn_01x02
- removed LBUCK1: 47µH, Inductor_SMD:L_Vishay_IHLP-4040, symbol Device:L
- removed LDO1: LMS8117, Package_TO_SOT_SMD:SOT-223-3_TabPin2, symbol LDO:LMS8117
- removed LED1, LED2: LED, LED_THT:LED_D3.0mm, symbol Device:LED
- removed MOTOR1: Conn_01x03, TerminalBlock_Phoenix:TerminalBlock_Phoenix_MKDS-1,5-3-5.08_1x03_P5.08mm_Horizontal, symbol Connector_Generic:Conn_01x03
- removed RCCOMP1, RCCOMP2, RFA1, RFB1, RFC1, RLED1, RLED2: R, Resistor_SMD:R_1206_3216Metric, symbol Device:R
Other:
- note removed: "INPUTS"
- note removed: "OUTPUTS"
- note removed: "R19 de alrededor 100 - 150Ω I_max_LED = 120mA"
- note removed: "Valores de R16, R17 y R18 altos ya que solo se necesita el voltaje comun"
