File: TM4C123GXL.kicad_sch (KiCad schematic)
At the start: 4 parts

Commit message: Guardar cambios
Parts:
- removed POT1: Conn_01x03, TerminalBlock_Phoenix:TerminalBlock_Phoenix_MKDS-1,5-3-5.08_1x03_P5.08mm_Horizontal, symbol Connector_Generic:Conn_01x03
- removed SPI1: Conn_01x07, Connector_PinHeader_2.54mm:PinHeader_1x07_P2.54mm_Vertical, symbol Connector_Generic:Conn_01x07
- removed TIVA13, TIVA42: Conn_02x10_Top_Bottom, Connector_PinSocket_2.54mm:PinSocket_2x10_P2.54mm_Vertical, symbol Connector_Generic:Conn_02x10_Top_Bottom
Other:
- note removed: "ADC"
- note removed: "BEMF_FASE_A"
- note removed: "BEMF_FASE_B"
- note removed: "BEMF_FASE_C"
- note removed: "LI_FASE_A"
- note removed: "LI_FASE_B"
- note removed: "LI_FASE_C"
- note removed: "MISO"
- note removed: "MOSI"
- note removed: "PMW_FASE_A"
- note removed: "PWM_FASE_B"
- note removed: "PWM_FASE_C"
- note removed: "SCLK"
- note removed: "SS1"
