File: Control Motor BLDC.kicad_pcb (KiCad board)
At the start: 4 copper layers, 70 x 90 mm, 94 parts

Commit message: Add files via upload
Parts:
- added BEMF_A: Conn_01x01, Connector_PinSocket_2.54mm:PinSocket_1x01_P2.54mm_Vertical, F.Cu at (124.3, 129.6)
- added BEMF_B: Conn_01x01, Connector_PinSocket_2.54mm:PinSocket_1x01_P2.54mm_Vertical, F.Cu at (120.6, 129.6)
- added BEMF_C: Conn_01x01, Connector_PinSocket_2.54mm:PinSocket_1x01_P2.54mm_Vertical, F.Cu at (116.9, 129.6)
- added TEST_5V: Conn_01x01, Connector_PinSocket_2.54mm:PinSocket_1x01_P2.54mm_Vertical, F.Cu at (85.8, 63.9)
- added TEST_COMPFA1: Conn_01x01, Connector_PinSocket_2.54mm:PinSocket_1x01_P2.54mm_Vertical, F.Cu at (111.5, 111.6)
- added TEST_COMPFB1: Conn_01x01, Connector_PinSocket_2.54mm:PinSocket_1x01_P2.54mm_Vertical, F.Cu at (115.2, 111.6)
- added TEST_COMPFC1: Conn_01x01, Connector_PinSocket_2.54mm:PinSocket_1x01_P2.54mm_Vertical, F.Cu at (118.9, 111.6)
- added TEST_COMPIN1: Conn_01x01, Connector_PinSocket_2.54mm:PinSocket_1x01_P2.54mm_Vertical, F.Cu at (122.6, 111.6)
- added V_n: Conn_01x01, Connector_PinSocket_2.54mm:PinSocket_1x01_P2.54mm_Vertical, F.Cu at (108.5, 52.8)
- moved TEST_BLDC1 15.8 mm to (145.3, 52.3)
- moved RFA1 15.8 mm to (140.1, 56.6)
- moved RFB1 15.8 mm to (142.7, 56.6)
- moved RFC1 15.8 mm to (145.3, 56.7)
- moved MOTOR1 15.0 mm to (130.2, 55.4)
- moved LED1 5.05 mm to (90.6, 63.9)
- moved RLED1 5.05 mm to (97.1, 63.9)
- moved RCCOMP1 3.26 mm to (107.0, 58.1)
Routing:
- net COMP_FA: track 62.3 -> 91.1 mm, vias 2 -> 5
- net +5V: track 0.00 -> 20.1 mm, vias 0 -> 1
- net N: track 23.6 -> 42.2 mm
- net COMP_FC: track 57.8 -> 73.1 mm, vias 2 -> 3
- net PD6: track 30.9 -> 44.7 mm
- net PD2: track 24.6 -> 37.4 mm, vias 1 -> 2
- net COMP_FB: track 58.5 -> 70.8 mm, vias 2 -> 5
- net FASE_C: track 53.5 -> 64.4 mm, vias 9 -> 11
- net COMP_IN: track 124.9 -> 133.3 mm, vias 7 -> 6
- net FASE_A: track 48.2 -> 40.0 mm
- net FASE_B: track 50.1 -> 42.3 mm
- net PD3: track 27.1 -> 34.7 mm
- net GND: track 176.1 -> 175.6 mm, vias 169 -> 166
- net VCC: vias 103 -> 99
- net +3V3: vias 28 -> 25
Other:
- board text added: "Phase A"
- board text added: "Phase B"
- board text added: "Phase C"

Commit message: corrijo errores
Parts:
- removed TEST_3V3, TEST_POT1, TEST_VBA1, TEST_VBB1, TEST_VBC1: Conn_01x01, Connector_PinSocket_2.54mm:PinSocket_1x01_P2.54mm_Vertical
- removed TEST_GA1, TEST_GB1, TEST_GC1, TEST_IA1, TEST_IB1, TEST_IC1: Conn_01x03, Connector_PinSocket_2.54mm:PinSocket_1x03_P2.54mm_Vertical
- added TST_3V3: Conn_01x01, Connector_PinSocket_2.54mm:PinSocket_1x01_P2.54mm_Vertical, F.Cu at (145.9, 125.6)
- added TST_GA1: Conn_01x03, Connector_PinSocket_2.54mm:PinSocket_1x03_P2.54mm_Vertical, F.Cu at (134.9, 66.2)
- added TST_GB1: Conn_01x03, Connector_PinSocket_2.54mm:PinSocket_1x03_P2.54mm_Vertical, F.Cu at (119.2, 66.2)
- added TST_GC1: Conn_01x03, Connector_PinSocket_2.54mm:PinSocket_1x03_P2.54mm_Vertical, F.Cu at (104.0, 66.5)
- added TST_IA1: Conn_01x03, Connector_PinSocket_2.54mm:PinSocket_1x03_P2.54mm_Vertical, F.Cu at (144.8, 101.0)
- added TST_IB1: Conn_01x03, Connector_PinSocket_2.54mm:PinSocket_1x03_P2.54mm_Vertical, F.Cu at (127.8, 100.8)
- added TST_IC1: Conn_01x03, Connector_PinSocket_2.54mm:PinSocket_1x03_P2.54mm_Vertical, F.Cu at (113.3, 100.8)
- added TST_POT1: Conn_01x01, Connector_PinSocket_2.54mm:PinSocket_1x01_P2.54mm_Vertical, F.Cu at (81.9, 128.4)
- added TST_VBA1: Conn_01x01, Connector_PinSocket_2.54mm:PinSocket_1x01_P2.54mm_Vertical, F.Cu at (134.8, 88.3)
- added TST_VBB1: Conn_01x01, Connector_PinSocket_2.54mm:PinSocket_1x01_P2.54mm_Vertical, F.Cu at (119.1, 88.1)
- added TST_VBC1: Conn_01x01, Connector_PinSocket_2.54mm:PinSocket_1x01_P2.54mm_Vertical, F.Cu at (104.0, 87.7)
- added TST_VCC1: Conn_01x01, Connector_PinSocket_2.54mm:PinSocket_1x01_P2.54mm_Vertical, F.Cu at (104.5, 52.9)
- moved FUENTE1 0.28 mm to (81.6, 101.5)
- moved LED2 0.17 mm to (145.9, 122.2)
- renumbered BEMF_A to BEMF_FA1, BEMF_B to BEMF_FB1, BEMF_C to BEMF_FC1, TEST_COMPFA1 to TEST_CFA1, TEST_COMPFB1 to TEST_CFB1, TEST_COMPFC1 to TEST_CFC1, TEST_5V to TST_5V1, V_n to V_N1
Routing:
- net COMP_FC: track 73.1 -> 71.3 mm
- net COMP_IN: track 133.3 -> 132.1 mm
- net COMP_FB: track 70.8 -> 71.2 mm, vias 5 -> 4
- net VCC: vias 99 -> 97
- net +3V3: vias 25 -> 28
Other:
- board text removed: "LMS8117"

Commit message: Corrijo errores de la placa (0 errors, 0 warnings)
Parts:
- removed TEST_CFA1, TEST_CFB1, TEST_CFC1, TEST_COMPIN1: Conn_01x01, Connector_PinSocket_2.54mm:PinSocket_1x01_P2.54mm_Vertical
- added CDC1: C, Capacitor_SMD:C_1206_3216Metric, F.Cu at (113.9, 122.4)
- added CIBUCK2: C, Capacitor_SMD:C_1206_3216Metric, B.Cu at (94.3, 87.0)
- added RCH1: R, Resistor_SMD:R_1206_3216Metric, B.Cu at (120.0, 127.3)
- added RCH2: R, Resistor_SMD:R_1206_3216Metric, F.Cu at (120.0, 127.3)
- added RCH3: R, Resistor_SMD:R_1206_3216Metric, F.Cu at (106.5, 122.9)
- added TST_CFA1: Conn_01x01, Connector_PinSocket_2.54mm:PinSocket_1x01_P2.54mm_Vertical, F.Cu at (111.5, 111.6)
- added TST_CFB1: Conn_01x01, Connector_PinSocket_2.54mm:PinSocket_1x01_P2.54mm_Vertical, F.Cu at (115.2, 111.6)
- added TST_CFC1: Conn_01x01, Connector_PinSocket_2.54mm:PinSocket_1x01_P2.54mm_Vertical, F.Cu at (118.9, 111.6)
- added TST_CIN1: Conn_01x01, Connector_PinSocket_2.54mm:PinSocket_1x01_P2.54mm_Vertical, F.Cu at (122.6, 111.6)
- moved RPC1 2.30 mm to (106.5, 122.9)
- moved BEMF_FB1 1.65 mm to (120.7, 131.2)
- moved BEMF_FA1 1.65 mm to (124.3, 131.2)
- moved BEMF_FC1 1.65 mm to (117.0, 131.2)
Connections:
- COMP1 pad 10: unconnected-(COMP1C---Pad10) -> +3V3
- COMP1 pad 11: unconnected-(COMP1C-+-Pad11) -> GND
- TIVA13 pad 14: IBH -> PD1
- TIVA13 pad 5: PE4 -> IBH
Routing:
- net PD6: track 44.7 -> 55.4 mm
- net COMP_FC: track 71.3 -> 78.1 mm
- net COMP_FB: track 71.2 -> 76.6 mm
- net COMP_FA: track 91.1 -> 96.2 mm
- net GND: track 175.6 -> 180.1 mm, vias 166 -> 167
- net IBH: track 30.2 -> 33.9 mm
- net PD3: track 34.7 -> 38.3 mm
- net PD2: track 37.4 -> 39.1 mm
- net PA5: track 29.2 -> 27.7 mm
- net PA4: track 28.8 -> 27.5 mm
- net +3V3: track 0.33 -> 0.18 mm, vias 28 -> 26
- net VCC: vias 97 -> 95

Commit message: Placa final (pre-revisión)
Parts:
- LBUCK1: footprint Inductor_SMD:L_Vishay_IHLP-4040 -> Inductor:Inductor
- moved FUENTE1 0.80 mm to (81.5, 102.3)
- moved LDO1 0.80 mm to (88.6, 103.5)
- moved DBUCK1 0.64 mm to (96.7, 92.5)
- moved LBUCK1 0.63 mm to (86.4, 93.3), turned to -90 degrees
Connections:
- SPI1 pad 3: PA5 -> PA3
- SPI1 pad 7: PF1 -> PA5
Routing:
- net PA3: track 0.00 -> 22.3 mm
- net VCC: track 21.1 -> 41.8 mm, vias 95 -> 103
- net PF1: track 13.4 -> 0.42 mm
- net PA5: track 27.9 -> 17.4 mm
- net GND: track 180.1 -> 177.2 mm, vias 167 -> 165
- net FASE_B: track 42.3 -> 43.0 mm
Other:
- board text added: "Universidad de Barcelona Argibay Molina Manuel Perez Pique Max"
