File: Control Motor BLDC.kicad_sch (KiCad schematic)
At the start: 0 parts

Commit message: Guardar cambios
Parts:
- added 12VIN1: Conn_01x02, TerminalBlock_Phoenix:TerminalBlock_Phoenix_MKDS-1,5-2-5.08_1x02_P5.08mm_Horizontal, symbol Connector_Generic:Conn_01x02
- added BUCK1: AP1509-50SG-13, Package_SO:SOP-8_3.76x4.96mm_P1.27mm, symbol AP1509:AP1509-50SG-13
- added CIBUCK1, COBUCK1: C_Polarized, Capacitor_SMD:CP_Elec_8x6.2, symbol Device:C_Polarized
- added CILDO1, COLDO1: C_Polarized, Capacitor_SMD:C_1206_3216Metric, symbol Device:C_Polarized
- added CIN1: C, Capacitor_SMD:CP_Elec_8x6.2, symbol Device:C
- added DBUCK1: B220, Diode_SMD:D_SMB, symbol Diode:B220
- added FUENTE1, TIVA1: Conn_01x02, Connector_PinHeader_2.54mm:PinHeader_1x02_P2.54mm_Vertical, symbol Connector_Generic:Conn_01x02
- added LBUCK1: 47µH, Inductor_SMD:L_Vishay_IHLP-4040, symbol Device:L
- added LDO1: LMS8117, Package_TO_SOT_SMD:SOT-223-3_TabPin2, symbol LDO:LMS8117
- added LED1, LED2: LED, LED_THT:LED_D3.0mm, symbol Device:LED
- added MOTOR1, POT1: Conn_01x03, TerminalBlock_Phoenix:TerminalBlock_Phoenix_MKDS-1,5-3-5.08_1x03_P5.08mm_Horizontal, symbol Connector_Generic:Conn_01x03
- added RCCOMP1, RCCOMP2, RFA1, RFB1, RFC1, RLED1, RLED2: R, Resistor_SMD:R_1206_3216Metric, symbol Device:R
- added SPI1: Conn_01x07, Connector_PinHeader_2.54mm:PinHeader_1x07_P2.54mm_Vertical, symbol Connector_Generic:Conn_01x07
- added TIVA13, TIVA42: Conn_02x10_Top_Bottom, Connector_PinSocket_2.54mm:PinSocket_2x10_P2.54mm_Vertical, symbol Connector_Generic:Conn_02x10_Top_Bottom
Connections:
- new net +3V3: FUENTE1.2 (Pin_2), POT1.1 (Pin_1), TIVA1.1 (Pin_1)
- new net +5V: BUCK1.3 (FB), CILDO1.1, COBUCK1.1, LBUCK1.2, LDO1.3 (Vin)
- new net +VBUS: TIVA13.11 (Pin_11)
- new net BUCK_OUT: BUCK1.2 (OUTPUT), DBUCK1.1 (K), LBUCK1.1
- new net COMP_IN: RCCOMP1.2, RCCOMP2.1
- new net FASE_A: MOTOR1.1 (Pin_1), RFA1.1
- new net FASE_B: MOTOR1.2 (Pin_2), RFB1.1
- new net FASE_C: MOTOR1.3 (Pin_3), RFC1.1
- new net GND: 12VIN1.2 (Pin_2), BUCK1.4 (SD), BUCK1.5 (GND_1), BUCK1.6 (GND_2), BUCK1.7 (GND_3), BUCK1.8 (GND_4), CIBUCK1.2, CILDO1.2, CIN1.2, COBUCK1.2, COLDO1.2, DBUCK1.2 (A), LDO1.1 (GND), LED1.1 (K), LED2.1 (K), POT1.3 (Pin_3), RCCOMP2.2, SPI1.2 (Pin_2), SPI1.4 (Pin_4), SPI1.6 (Pin_6), TIVA13.12 (Pin_12), TIVA42.1 (Pin_1)
- new net LDO_+3V3: COLDO1.1, FUENTE1.1 (Pin_1), LDO1.2 (Vout)
- new net LED2_IN: LED2.2 (A), RLED2.2
- new net LED_IN: LED1.2 (A), RLED1.2
- new net N: RCCOMP1.1, RFA1.2, RFB1.2, RFC1.2
- new net PA2: SPI1.1 (Pin_1), TIVA42.10 (Pin_10)
- new net PA3: TIVA42.9 (Pin_9)
- new net PA4: SPI1.5 (Pin_5), TIVA42.8 (Pin_8)
- new net PA5: SPI1.3 (Pin_3), TIVA13.8 (Pin_8)
- new net PA6: TIVA13.9 (Pin_9)
- new net PA7: TIVA13.10 (Pin_10)
- new net PB0: TIVA13.3 (Pin_3)
- new net PB1: TIVA13.4 (Pin_4)
- new net PB2: TIVA42.2 (Pin_2)
- new net PB3: TIVA42.13 (Pin_13)
- new net PB4: TIVA13.7 (Pin_7)
- new net PB5: TIVA13.2 (Pin_2)
- new net PB6: TIVA42.7 (Pin_7)
- new net PB7: TIVA42.6 (Pin_6)
- new net PC5: TIVA42.15 (Pin_15)
- new net PC6: TIVA42.16 (Pin_16)
- new net PC7: TIVA42.17 (Pin_17)
- new net PD0: TIVA13.13 (Pin_13)
- new net PD1: TIVA13.14 (Pin_14)
- new net PD2: TIVA13.15 (Pin_15)
- new net PD3: TIVA13.16 (Pin_16)
- new net PD6: TIVA42.18 (Pin_18)
- new net PD7: TIVA42.19 (Pin_19)
- new net PE0: POT1.2 (Pin_2), TIVA42.3 (Pin_3)
- new net PE1: TIVA13.17 (Pin_17)
- new net PE2: TIVA13.18 (Pin_18)
- new net PE3: TIVA13.19 (Pin_19)
- new net PE4: TIVA13.5 (Pin_5)
- new net PE5: TIVA13.6 (Pin_6)
- new net PF0: TIVA42.4 (Pin_4)
- new net PF1: SPI1.7 (Pin_7), TIVA13.20 (Pin_20)
- new net PF2: TIVA42.11 (Pin_11)
- new net PF3: TIVA42.12 (Pin_12)
- new net PF4: TIVA42.20 (Pin_20)
- new net TIVA_+3V3: RLED2.1, TIVA1.2 (Pin_2), TIVA13.1 (Pin_1)
- new net VCC: 12VIN1.1 (Pin_1), BUCK1.1 (VIN), CIBUCK1.1, CIN1.1, RLED1.1
- new net /TARGETRST: TIVA42.5 (Pin_5)
Other:
- removed sheet Inputs y Outputs
- removed sheet TM4C123GXL
- note added: "3.3V switch (Buck-LDO or TIVA-C)"
- note added: "ADC"
- note added: "BEMF_FASE_A"
- note added: "BEMF_FASE_B"
- note added: "BEMF_FASE_C"
- note added: "Buck structure (12V to 5V conversion)"
- note added: "INPUTS/OUTPUTS"
- note added: "LDO structure (5V to 3.3V conversion)"
- note added: "LI_FASE_A"
- note added: "LI_FASE_B"
- note added: "LI_FASE_C"
- note added: "MISO"
- note added: "MOSI"
- note added: "Motor Connector & V_n extract"
- note added: "PMW_FASE_A"
- note added: "POWER"
- note added: "PWM_FASE_B"
- note added: "PWM_FASE_C"
- note added: "Potentiometer Connector"
- note added: "R19 de alrededor 100 - 150Ω I_max_LED = 120mA"
- note added: "SCLK"
- note added: "SPI Connector"
- note added: "SS1"
- note added: "TIVA-C connectors"
- note added: "VCC Connector"
- note added: "Valores de R16, R17 y R18 altos ya que solo se necesita el voltaje comun"
- note removed: "INPUTS Y OUTPUTS"
- note removed: "TIVA-TM4C123GXL"
- company: (none) -> Universitat de Barcelona
- title: (none) -> Placa LSE Manu & Max

Commit message: Update proyecto KiCad - revision esquematico
Parts:
- added BEMF_FaseA1, BEMF_FaseB1, BEMF_FaseC1, TEST_3V3, TEST_5V1, TEST_COMPFA1, TEST_COMPFB1, TEST_COMPFC1, TEST_COMPIN1, TEST_POT1, TEST_VBA1, TEST_VBB1, TEST_VBC1, TEST_VCC1, V_n1: Conn_01x01, Connector_PinSocket_2.54mm:PinSocket_1x01_P2.54mm_Vertical, symbol Connector_Generic:Conn_01x01
- added CA1, CB1, CBA1, CBB1, CBC1, CC1, CCA1, CCB1, CCC1, CDAH1, CDBH1, CDCH1, CIAH1, CIAL1, CIBH1, CIBL1, CICH1, CICL1: C, Capacitor_SMD:C_1206_3216Metric, symbol Device:C
- added COMP1: LM339, Package_SO:SOIC-14_3.9x8.7mm_P1.27mm, symbol Comparator:LM339
- added DA1, DB1, DC1: IR2301, Package_SO:SOIC-8_3.9x4.9mm_P1.27mm, symbol Driver_FET:IR2301
- added DBA1, DBB1, DBC1: 1N4149, Diode_THT:D_DO-35_SOD27_P7.62mm_Horizontal, symbol Diode:1N4149
- added MAH1, MAL1, MBH1, MBL1, MCH1, MCL1: NMOS, NMOS:NMOS, symbol Simulation_SPICE:NMOS
- added RC1A1, RC1B1, RC1C1, RC2A1, RC2B1, RC2C1, RGAH1, RGAL1, RGBH1, RGBL1, RGCH1, RGCL1, RIAH1, RIAL1, RIBH1, RIBL1, RICH1, RICL1, RPA1, RPB1, RPC1: R, Resistor_SMD:R_1206_3216Metric, symbol Device:R
- added TEST_BLDC1: Conn_01x04, Connector_PinHeader_2.54mm:PinHeader_1x04_P2.54mm_Vertical, symbol Connector_Generic:Conn_01x04
- added TEST_GA1, TEST_GB1, TEST_GC1, TEST_IA1, TEST_IB1, TEST_IC1: Conn_01x03, Connector_PinSocket_2.54mm:PinSocket_1x03_P2.54mm_Vertical, symbol Connector_Generic:Conn_01x03
Connections:
- net +3V3: now also COMP1.3 (V+), RPA1.1, RPB1.1, RPC1.1, TEST_3V3.1 (Pin_1)
- net +5V: now also TEST_5V1.1 (Pin_1)
- net COMP_IN: now also CCA1.2, CCB1.2, CCC1.2, COMP1.4 (-), COMP1.6 (-), COMP1.8 (-), TEST_COMPIN1.1 (Pin_1)
- net FASE_A: now also CBA1.2, DA1.6 (VS), MAH1.3 (S), MAL1.1 (D), RC1A1.1, TEST_BLDC1.3 (Pin_3)
- net FASE_B: now also CBB1.2, DB1.6 (VS), MBH1.3 (S), MBL1.1 (D), RC1B1.1, TEST_BLDC1.2 (Pin_2)
- net FASE_C: now also CBC1.2, DC1.6 (VS), MCH1.3 (S), MCL1.1 (D), RC1C1.1, TEST_BLDC1.1 (Pin_1)
- net GND: now also CA1.2, CB1.1, CC1.1, CDAH1.2, CDBH1.2, CDCH1.2, CIAH1.1, CIAL1.1, CIBH1.1, CIBL1.1, CICH1.1, CICL1.1, COMP1.12 (V-), DA1.4 (COM), DB1.4 (COM), DC1.4 (COM), MAL1.3 (S), MBL1.3 (S), MCL1.3 (S), RC2A1.2, RC2B1.2, RC2C1.2, TEST_BLDC1.4 (Pin_4), TEST_GA1.3 (Pin_3), TEST_GB1.3 (Pin_3), TEST_GC1.3 (Pin_3), TEST_IA1.3 (Pin_3), TEST_IB1.3 (Pin_3), TEST_IC1.3 (Pin_3)
- net N: now also V_n1.1 (Pin_1)
- net PC4: now also TIVA42.14 (Pin_14)
- net PD2: now also BEMF_FaseB1.1 (Pin_1), COMP1.1, RPB1.2
- net PD3: now also BEMF_FaseA1.1 (Pin_1), COMP1.2, RPA1.2
- net PD6: now also BEMF_FaseC1.1 (Pin_1), COMP1.14, RPC1.2
- net PE0: now also TEST_POT1.1 (Pin_1)
- net VCC: now also CA1.1, CB1.2, CC1.2, CDAH1.1, CDBH1.1, CDCH1.1, DA1.1 (VCC), DB1.1 (VCC), DBA1.2 (A), DBB1.2 (A), DBC1.2 (A), DC1.1 (VCC), MAH1.1 (D), MBH1.1 (D), MCH1.1 (D), TEST_VCC1.1 (Pin_1)
- net PB3 renamed IBL
- net IBL: now also RIBL1.1, TEST_IB1.2 (Pin_2)
- net PB5 renamed IAH
- net IAH: now also RIAH1.1, TEST_IA1.1 (Pin_1)
- net PB7 renamed ICH
- net ICH: now also RICH1.1, TEST_IC1.1 (Pin_1)
- net PD0 renamed IAL
- net IAL: now also RIAL1.1, TEST_IA1.2 (Pin_2)
- net PD1 renamed IBH
- net IBH: now also RIBH1.1, TEST_IB1.1 (Pin_1)
- net PF2 renamed ICL
- net ICL: now also RICL1.1, TEST_IC1.2 (Pin_2)
- new net AHIN: CIAH1.2, DA1.2 (HIN), RIAH1.2
- new net ALIN: CIAL1.2, DA1.3 (LIN), RIAL1.2
- new net BHIN: CIBH1.2, DB1.2 (HIN), RIBH1.2
- new net BLIN: CIBL1.2, DB1.3 (LIN), RIBL1.2
- new net CHIN: CICH1.2, DC1.2 (HIN), RICH1.2
- new net CLIN: CICL1.2, DC1.3 (LIN), RICL1.2
- new net COMP_FA: CCA1.1, COMP1.5 (+), RC1A1.2, RC2A1.1, TEST_COMPFA1.1 (Pin_1)
- new net COMP_FB: CCB1.1, COMP1.7 (+), RC1B1.2, RC2B1.1, TEST_COMPFB1.1 (Pin_1)
- new net COMP_FC: CCC1.1, COMP1.9 (+), RC1C1.2, RC2C1.1, TEST_COMPFC1.1 (Pin_1)
- new net GAH: MAH1.2 (G), RGAH1.2, TEST_GA1.1 (Pin_1)
- new net GAL: MAL1.2 (G), RGAL1.1, TEST_GA1.2 (Pin_2)
- new net GBH: MBH1.2 (G), RGBH1.2, TEST_GB1.1 (Pin_1)
- new net GBL: MBL1.2 (G), RGBL1.1, TEST_GB1.2 (Pin_2)
- new net GCH: MCH1.2 (G), RGCH1.2, TEST_GC1.1 (Pin_1)
- new net GCL: MCL1.2 (G), RGCL1.1, TEST_GC1.2 (Pin_2)
- new net HOA: DA1.7 (HO), RGAH1.1
- new net HOB: DB1.7 (HO), RGBH1.1
- new net HOC: DC1.7 (HO), RGCH1.1
- new net LOA: DA1.5 (LO), RGAL1.2
- new net LOB: DB1.5 (LO), RGBL1.2
- new net LOC: DC1.5 (LO), RGCL1.2
- new net VBA: CBA1.1, DA1.8 (VB), DBA1.1 (K), TEST_VBA1.1 (Pin_1)
- new net VBB: CBB1.1, DB1.8 (VB), DBB1.1 (K), TEST_VBB1.1 (Pin_1)
- new net VBC: CBC1.1, DBC1.1 (K), DC1.8 (VB), TEST_VBC1.1 (Pin_1)
- no-connect marks 0 -> 3
Other:
- removed sheet Motor
- removed sheet Testpoints
- note added: "3 (one for each phase) - Half-fridge structure"
- note added: "BEMF_FASE1"
- note added: "BEMF_FASE2"
- note added: "BEMF_FASE3"
- note added: "Half-bridge (A)"
- note added: "Half-bridge (B)"
- note added: "Half-bridge (C)"
- note added: "Motor BLDC"
- note added: "PMW_FASE_B"
- note added: "PMW_FASE_C"
- note added: "Phase A"
- note added: "Phase B"
- note added: "Phase C"
- note added: "Potentiometer"
- note added: "Power"
- note added: "V_n extraction"
- note added: "Zero-pass detector + BEMF network"
- note removed: "MOTOR, DRIVERS Y CONTROL"

Commit message: corrijo errores
Parts:
- renumbered BEMF_FaseA1 to BEMF_FA1, BEMF_FaseB1 to BEMF_FB1, BEMF_FaseC1 to BEMF_FC1, TEST_COMPFA1 to TEST_CFA1, TEST_COMPFB1 to TEST_CFB1, TEST_COMPFC1 to TEST_CFC1, TEST_3V3 to TST_3V3, TEST_5V1 to TST_5V1, TEST_GA1 to TST_GA1, TEST_GB1 to TST_GB1, TEST_GC1 to TST_GC1, TEST_IA1 to TST_IA1, TEST_IB1 to TST_IB1, TEST_IC1 to TST_IC1, TEST_POT1 to TST_POT1, TEST_VBA1 to TST_VBA1, TEST_VBB1 to TST_VBB1, TEST_VBC1 to TST_VBC1, TEST_VCC1 to TST_VCC1, V_n1 to V_N1
Changed lines of the file:
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@@
 		(on_board yes)
 		(dnp no)
-		(property "Reference" "TEST_COMPFB1"
+		(property "Reference" "TEST_CFB1"
 			(at 342.646 237.49 0)
 			(effects
@@
 			(project "Control Motor BLDC"
 				(path "/dcdea0bb-21d8-4b74-9d07-c2aa983143bc"
-					(reference "TEST_COMPFB1")
+					(reference "TEST_CFB1")
 					(unit 1)
 				)
@@
 		(on_board yes)
 		(dnp no)
-		(property "Reference" "TEST_3V3"
+		(property "Reference" "TST_3V3"
 			(at 138.176 264.16 0)
 			(effects
@@
 			(project "Control Motor BLDC"
 				(path "/dcdea0bb-21d8-4b74-9d07-c2aa983143bc"
-					(reference "TEST_3V3")
+					(reference "TST_3V3")
 					(unit 1)
 				)
@@
 		(dnp no)
 		(fields_autoplaced yes)
-		(property "Reference" "TEST_GB1"
+		(property "Reference" "TST_GB1"
 			(at 205.74 242.5699 0)
 			(effects
@@
 			(project "Control Motor BLDC"
 				(path "/dcdea0bb-21d8-4b74-9d07-c2aa983143bc"
-					(reference "TEST_GB1")
+					(reference "TST_GB1")
 					(unit 1)
 				)
@@
 		(on_board yes)
 		(dnp no)
-		(property "Reference" "TEST_VCC1"
+		(property "Reference" "TST_VCC1"
 			(at 138.176 246.38 0)
 			(effects
@@
 			(project "Control Motor BLDC"
 				(path "/dcdea0bb-21d8-4b74-9d07-c2aa983143bc"
-					(reference "TEST_VCC1")
+					(reference "TST_VCC1")
 					(unit 1)
 				)
@@
 		(on_board yes)
 		(dnp no)
-		(property "Reference" "TEST_VBB1"
+		(property "Reference" "TST_VBB1"
 			(at 202.946 274.32 0)
 			(effects
@@
 			(project "Control Motor BLDC"
 				(path "/dcdea0bb-21d8-4b74-9d07-c2aa983143bc"
-					(reference "TEST_VBB1")
+					(reference "TST_VBB1")
 					(unit 1)
 				)
@@
 		(on_board yes)
 		(dnp no)
-		(property "Reference" "TEST_POT1"
+		(property "Reference" "TST_POT1"
 			(at 267.716 280.67 0)
 			(effects
@@
 			(project "Control Motor BLDC"
 				(path "/dcdea0bb-21d8-4b74-9d07-c2aa983143bc"
-					(reference "TEST_POT1")
+					(reference "TST_POT1")
 					(unit 1)
 				)
@@
 		(dnp no)
 		(fields_autoplaced yes)
-		(property "Reference" "TEST_IC1"
+		(property "Reference" "TST_IC1"
 			(at 236.22 261.6199 0)
 			(effects
@@
 			(project "Control Motor BLDC"
 				(path "/dcdea0bb-21d8-4b74-9d07-c2aa983143bc"
-					(reference "TEST_IC1")
+					(reference "TST_IC1")
 					(unit 1)
 				)
@@
 		(on_board yes)
 		(dnp no)
-		(property "Reference" "BEMF_FaseA1"
+		(property "Reference" "BEMF_FA1"
 			(at 305.816 246.38 0)
 			(effects
@@
 			(project "Control Motor BLDC"
 				(path "/dcdea0bb-21d8-4b74-9d07-c2aa983143bc"
-					(reference "BEMF_FaseA1")
+					(reference "BEMF_FA1")
 					(unit 1)
 				)
@@
 		(on_board yes)
 		(dnp no)
-		(property "Reference" "BEMF_FaseC1"
+		(property "Reference" "BEMF_FC1"
 			(at 384.556 245.11 0)
 			(effects
@@
 			(project "Control Motor BLDC"
 				(path "/dcdea0bb-21d8-4b74-9d07-c2aa983143bc"
-					(reference "BEMF_FaseC1")
+					(reference "BEMF_FC1")
 					(unit 1)
 				)
@@
 		(dnp no)
 		(fields_autoplaced yes)
-		(property "Reference" "TEST_IB1"
+		(property "Reference" "TST_IB1"
 			(at 205.74 261.6199 0)
 			(effects
@@
 			(project "Control Motor BLDC"
 				(path "/dcdea0bb-21d8-4b74-9d07-c2aa983143bc"
-					(reference "TEST_IB1")
+					(reference "TST_IB1")
 					(unit 1)
 				)
@@
 		(on_board yes)
 		(dnp no)
-		(property "Reference" "BEMF_FaseB1"
+		(property "Reference" "BEMF_FB1"
 			(at 342.646 246.38 0)
 			(effects
@@
 			(project "Control Motor BLDC"
 				(path "/dcdea0bb-21d8-4b74-9d07-c2aa983143bc"
-					(reference "BEMF_FaseB1")
+					(reference "BEMF_FB1")
 					(unit 1)
 				)
@@
 		(on_board yes)
 		(dnp no)
-		(property "Reference" "TEST_VBC1"
+		(property "Reference" "TST_VBC1"
 			(at 235.966 274.32 0)
 			(effects
@@
 			(project "Control Motor BLDC"
 				(path "/dcdea0bb-21d8-4b74-9d07-c2aa983143bc"
-					(reference "TEST_VBC1")
+					(reference "TST_VBC1")
 					(unit 1)
 				)
@@
 		(on_board yes)
 		(dnp no)
-		(property "Reference" "TEST_COMPFC1"
+		(property "Reference" "TEST_CFC1"
 			(at 384.556 237.49 0)
 			(effects
@@
 			(project "Control Motor BLDC"
 				(path "/dcdea0bb-21d8-4b74-9d07-c2aa983143bc"
-					(reference "TEST_COMPFC1")
+					(reference "TEST_CFC1")
 					(unit 1)
 				)
@@
 		(on_board yes)
 		(dnp no)
-		(property "Reference" "TEST_5V1"
+		(property "Reference" "TST_5V1"
 			(at 138.176 255.27 0)
 			(effects
@@
 			(project "Control Motor BLDC"
 				(path "/dcdea0bb-21d8-4b74-9d07-c2aa983143bc"
-					(reference "TEST_5V1")
+					(reference "TST_5V1")
 					(unit 1)
 				)
@@
 		(on_board yes)
 		(dnp no)
-		(property "Reference" "TEST_VBA1"
+		(property "Reference" "TST_VBA1"
 			(at 167.386 275.59 0)
 			(effects
@@
 			(project "Control Motor BLDC"
 				(path "/dcdea0bb-21d8-4b74-9d07-c2aa983143bc"
-					(reference "TEST_VBA1")
+					(reference "TST_VBA1")
 					(unit 1)
 				)
@@
 		(on_board yes)
 		(dnp no)
-		(property "Reference" "V_n1"
+		(property "Reference" "V_N1"
 			(at 266.446 260.35 0)
 			(effects
@@
 			(project "Control Motor BLDC"
 				(path "/dcdea0bb-21d8-4b74-9d07-c2aa983143bc"
-					(reference "V_n1")
+					(reference "V_N1")
 					(unit 1)
 				)
@@
 		(dnp no)
 		(fields_autoplaced yes)
-		(property "Reference" "TEST_GC1"
+		(property "Reference" "TST_GC1"
 			(at 236.22 242.5699 0)
 			(effects
@@
 			(project "Control Motor BLDC"
 				(path "/dcdea0bb-21d8-4b74-9d07-c2aa983143bc"
-					(reference "TEST_GC1")
+					(reference "TST_GC1")
 					(unit 1)
 				)
@@
 		(dnp no)
 		(fields_autoplaced yes)
-		(property "Reference" "TEST_GA1"
+		(property "Reference" "TST_GA1"
 			(at 168.91 241.2999 0)
 			(effects
@@
 			(project "Control Motor BLDC"
 				(path "/dcdea0bb-21d8-4b74-9d07-c2aa983143bc"
-					(reference "TEST_GA1")
+					(reference "TST_GA1")
 					(unit 1)
 				)
@@
 		(dnp no)
 		(fields_autoplaced yes)
-		(property "Reference" "TEST_IA1"
+		(property "Reference" "TST_IA1"
 			(at 168.91 260.3499 0)
 			(effects
@@
 			(project "Control Motor BLDC"
 				(path "/dcdea0bb-21d8-4b74-9d07-c2aa983143bc"
-					(reference "TEST_IA1")
+					(reference "TST_IA1")
 					(unit 1)
 				)
@@
 		(on_board yes)
 		(dnp no)
-		(property "Reference" "TEST_COMPFA1"
+		(property "Reference" "TEST_CFA1"
 			(at 304.546 237.49 0)
 			(effects
@@
 			(project "Control Motor BLDC"
 				(path "/dcdea0bb-21d8-4b74-9d07-c2aa983143bc"
-					(reference "TEST_COMPFA1")
+					(reference "TEST_CFA1")
 					(unit 1)
 				)

Commit message: Corrijo errores de la placa (0 errors, 0 warnings)
Parts:
- added CDC1, CIBUCK2: C, Capacitor_SMD:C_1206_3216Metric, symbol Device:C
- added RCH1, RCH2, RCH3: R, Resistor_SMD:R_1206_3216Metric, symbol Device:R
- renumbered TEST_CFA1 to TST_CFA1, TEST_CFB1 to TST_CFB1, TEST_CFC1 to TST_CFC1, TEST_COMPIN1 to TST_CIN1
Connections:
- net PE4 is gone; now on net IBH: TIVA13.5 (Pin_5)
- net +3V3: now also COMP1.10 (-), CDC1.1
- net COMP_FA: now also RCH1.1
- net COMP_FB: now also RCH2.1
- net COMP_FC: now also RCH3.1
- net GND: now also COMP1.11 (+), CDC1.2, CIBUCK2.2
- net IBH: no longer TIVA13.14 (Pin_14)
- net PD2: now also RCH2.2
- net PD3: now also RCH1.2
- net PD6: now also RCH3.2
- net VCC: now also CIBUCK2.1
- new net PD1: TIVA13.14 (Pin_14)
- no-connect marks 3 -> 1
Other:
- moved on the sheet: CIBUCK1, RPA1, RPB1, RPC1

Commit message: Commit
Other:
- note added: "In our BLDC motor, the neutral point is not accessible because the windings are internally connected. A virtual neutral is therefore generated to provide a reference voltage for the BEMF circuit to detect zero crossings"
- note added: "The BEMF circuit measures the back-electromotive force generated by the unpowered phase of the BLDC motor. The zero-crossing detector compares this signal with the virtual neutral voltage to identify zero crossings. This allows the rotor position to be estimated and the motor phases to be commutated at the correct time without position sensors."
- note added: "This LDO regulator provides a stable output voltage (3.3V) by regulating the input voltage with a low dropout voltage."
- note added: "This buck converter is a switched-mode step-down converter that converts the VCC input voltage to a stable 5 V output."
- note added: "This half-bridge stage uses two MOSFETs and a driver to control the switching of one phase (Phase A). The driver provides the required gate signals and dead time to ensure safe switching and prevent shoot-through"
- note added: "This half-bridge stage uses two MOSFETs and a driver to control the switching of one phase (Phase B)."
- note added: "This half-bridge stage uses two MOSFETs and a driver to control the switching of one phase (Phase C)."
- note added: "This structure allows us to choose between the 3.3 V supply from the TIVA-C or the Buck-LDO stage. Using both simultaneously could damage the circuit, as they are independent power sources."
- moved on the sheet: FUENTE1, LED2, MAL1, RLED2, TIVA1
