File: Control Motor BLDC.kicad_sch (KiCad schematic)
At the start: 105 parts

Commit message: Placa final (pre-revisión)
Parts:
- LBUCK1: footprint Inductor_SMD:L_Vishay_IHLP-4040 -> Inductor:Inductor
Connections:
- net PA3: now also SPI1.3 (Pin_3)
- net PA5: now also SPI1.7 (Pin_7); no longer SPI1.3 (Pin_3)
- net PF1: no longer SPI1.7 (Pin_7)
Changed lines of the file:
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@@
 	(text "SS1"
 		(exclude_from_sim no)
-		(at 314.198 65.278 0)
+		(at 368.808 64.008 0)
 		(effects
 			(font
@@
 	(text "SCLK"
 		(exclude_from_sim no)
-		(at 395.986 122.174 0)
+		(at 394.97 122.174 0)
 		(effects
 			(font
@@
 	(text "MOSI"
 		(exclude_from_sim no)
-		(at 394.716 127.508 0)
+		(at 394.716 137.414 0)
 		(effects
 			(font
@@
 	(text "LI_FASE_B"
 		(exclude_from_sim no)
-		(at 277.368 62.738 0)
+		(at 331.724 48.514 0)
 		(effects
 			(font
@@
 	(text "SS1"
 		(exclude_from_sim no)
-		(at 394.462 137.668 0)
+		(at 394.462 127.254 0)
 		(effects
 			(font
@@
 	(wire
 		(pts
-			(xy 339.09 123.19) (xy 340.36 123.19)
-		)
-		(stroke
-			(width 0)
-			(type default)
-			(color 0 255 0 1)
-		)
-	)
-	(wire
-		(pts
 			(xy 292.1 132.08) (xy 292.1 130.81)
 		)
@@
 	(wire
 		(pts
-			(xy 340.36 128.27) (xy 340.36 133.35)
+			(xy 345.44 128.27) (xy 345.44 133.35)
 		)
 		(stroke
@@
 	(wire
 		(pts
-			(xy 387.35 121.92) (xy 384.81 121.92)
+			(xy 386.08 121.92) (xy 384.81 121.92)
 		)
 		(stroke
@@
 	(wire
 		(pts
-			(xy 340.36 119.38) (xy 340.36 123.19)
+			(xy 345.44 119.38) (xy 345.44 123.19)
 		)
 		(stroke
@@
 	(wire
 		(pts
-			(xy 339.09 128.27) (xy 340.36 128.27)
+			(xy 339.09 128.27) (xy 345.44 128.27)
 		)
 		(stroke
@@
 		)
 	)
+	(wire
+		(pts
+			(xy 339.09 123.19) (xy 345.44 123.19)
+		)
+		(stroke
+			(width 0)
+			(type default)
+			(color 0 255 0 1)
+		)
+	)
 	(polyline
 		(pts
@@
 		)
 	)
-	(global_label "PA5"
-		(shape input)
-		(at 386.08 127 0)
-		(fields_autoplaced yes)
-		(effects
-			(font
-				(size 1.27 1.27)
-			)
-			(justify left)
-		)
-		(property "Intersheetrefs" "${INTERSHEET_REFS}"
-			(at 392.6333 127 0)
-			(effects
-				(font
-					(size 1.27 1.27)
-				)
-				(justify left)
-				(hide yes)
-			)
-		)
-	)
 	(global_label "PD2"
 		(shape input)
@@
 	(global_label "PA2"
 		(shape input)
-		(at 387.35 121.92 0)
+		(at 386.08 121.92 0)
 		(fields_autoplaced yes)
 		(effects
@@
 		)
 		(property "Intersheetrefs" "${INTERSHEET_REFS}"
-			(at 393.9033 121.92 0)
+			(at 392.6333 121.92 0)
 			(effects
 				(font
@@
 		)
 	)
+	(global_label "PA5"
+		(shape input)
+		(at 386.08 137.16 0)
+		(fields_autoplaced yes)
+		(effects
+			(font
+				(size 1.27 1.27)
+			)
+			(justify left)
+		)
+		(property "Intersheetrefs" "${INTERSHEET_REFS}"
+			(at 392.6333 137.16 0)
+			(effects
+				(font
+					(size 1.27 1.27)
+				)
+				(justify left)
+				(hide yes)
+			)
+		)
+	)
 	(global_label "PC4"
 		(shape input)
@@
 		)
 	)
-	(global_label "PF1"
-		(shape input)
-		(at 386.08 137.16 0)
-		(fields_autoplaced yes)
-		(effects
-			(font
-				(size 1.27 1.27)
-			)
-			(justify left)
-		)
-		(property "Intersheetrefs" "${INTERSHEET_REFS}"
-			(at 392.6333 137.16 0)
-			(effects
-				(font
-					(size 1.27 1.27)
-				)
-				(justify left)
-				(hide yes)
-			)
-		)
-	)
 	(global_label "PD2"
 		(shape input)
@@
 		)
 	)
+	(global_label "PA3"
+		(shape input)
+		(at 386.08 127 0)
+		(fields_autoplaced yes)
+		(effects
+			(font
+				(size 1.27 1.27)
+			)
+			(justify left)
+		)
+		(property "Intersheetrefs" "${INTERSHEET_REFS}"
+			(at 392.6333 127 0)
+			(effects
+				(font
+					(size 1.27 1.27)
+				)
+				(justify left)
+				(hide yes)
+			)
+		)
+	)
 	(global_label "PB0"
 		(shape input)
@@
 	(symbol
 		(lib_id "power:GND")
-		(at 340.36 133.35 0)
+		(at 345.44 133.35 0)
 		(unit 1)
 		(exclude_from_sim no)
@@
 		(fields_autoplaced yes)
 		(property "Reference" "#PWR013"
-			(at 340.36 139.7 0)
+			(at 345.44 139.7 0)
 			(effects
 				(font
@@
 		)
 		(property "Value" "GND"
-			(at 340.36 138.43 0)
+			(at 345.44 138.43 0)
 			(effects
 				(font
@@
 		)
 		(property "Footprint" ""
-			(at 340.36 133.35 0)
+			(at 345.44 133.35 0)
 			(effects
 				(font
@@
 		)
 		(property "Datasheet" ""
-			(at 340.36 133.35 0)
+			(at 345.44 133.35 0)
 			(effects
 				(font
@@
 		)
 		(property "Description" "Power symbol creates a global label with name \"GND\" , ground"
-			(at 340.36 133.35 0)
+			(at 345.44 133.35 0)
 			(effects
 				(font
@@
 			)
 		)
-		(property "Footprint" "Inductor_SMD:L_Vishay_IHLP-4040"
+		(property "Footprint" "Inductor:Inductor"
 			(at 99.06 46.99 0)
 			(effects
@@
 	(symbol
 		(lib_id "power:+3V3")
-		(at 340.36 119.38 0)
+		(at 345.44 119.38 0)
 		(unit 1)
 		(exclude_from_sim no)
@@
 		(fields_autoplaced yes)
 		(property "Reference" "#PWR012"
-			(at 340.36 123.19 0)
+			(at 345.44 123.19 0)
 			(effects
 				(font
@@
 		)
 		(property "Value" "+3V3"
-			(at 340.36 114.3 0)
+			(at 345.44 114.3 0)
 			(effects
 				(font
@@
 		)
 		(property "Footprint" ""
-			(at 340.36 119.38 0)
+			(at 345.44 119.38 0)
 			(effects
 				(font
@@
 		)
 		(property "Datasheet" ""
-			(at 340.36 119.38 0)
+			(at 345.44 119.38 0)
 			(effects
 				(font
@@
 		)
 		(property "Description" "Power symbol creates a global label with name \"+3V3\""
-			(at 340.36 119.38 0)
+			(at 345.44 119.38 0)
 			(effects
 				(font
